File: mPCIE-to-M_2_E-Key.kicad_sch (KiCad schematic)
At the start: 11 parts, among them J1 Bus_PCI_Express_Mini, J2 Bus_M.2_Socket_E, Q1 BSS138K, Q2 BSS138K, U1 TL1963A

Commit message: updated files
Parts:
- removed U1: TL1963A, lib_fp:SOT223-4, symbol lib_sch:TL1963A-XX
- added H1, H2: M2.5, lib_fp:M2.5_MH, symbol Mechanical:MountingHole_Pad
- added H3: M3.5, lib_fp:MountingHole_3.5mm_Pad_Via, symbol Mechanical:MountingHole_Pad
- added R5: 100K, lib_fp:CRCW0603, symbol lib_sch:R
- added U1: TPS79718, lib_fp:SOT323-65P210X110-5, symbol lib_sch:TPS797xx-Q1
- C1: value 10uF -> 100nF; footprint lib_fp:CAPC160X80X88L35N -> lib_fp:MLCC0603; DKPN 478-KGM15CR51E106KTCT-ND -> 478-KAM15AR71H104KMCT-ND; MPN 06033D106KAT2A -> 06035C104K4T4A; Voltage Rating 25V -> 50V
- C2: value 10uF -> 470nF; footprint lib_fp:CAPC160X80X88L35N -> lib_fp:MLCC0805; DKPN 478-KGM15CR51E106KTCT-ND -> 478-KAM21KR71C474KUCT-ND; MPN 06033D106KAT2A -> KAM21KR71C474KU; Package 0603 -> 0805; Voltage Rating 25V -> 16V
- J1: footprint (none) -> lib_fp:BUS_mPCIe
- R1, R2, R3, R4: footprint lib_fp:RESC160X80X55L30N -> lib_fp:CRCW0603
Connections:
- net +1V8: now also R5.1, U1.5 (OUT)
- net +3V3: now also U1.4 (IN)
- net GND: now also J2.S1 (MP), J2.S2 (MP), H1.1, H2.1, H3.1, U1.2 (GND); no longer J1.MP
- net SCL_1V8: now also Q1.2, R3.2
- net SCL_3V3: now also Q1.3, R1.2
- net SDA_1V8: now also Q2.2, R4.2
- net SDA_3V3: now also Q2.3, R2.2
- new net: R5.2, U1.1 (PG)
- no-connect marks 73 -> 75
Other:
- moved on the sheet: C2

Commit message: fixed 1V8 reg DKPN
Parts:
- U1: DKPN 296-23648-6-ND -> 296-23648-1-ND
Changed lines of the file:
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@@
 			)
 		)
-		(property "DKPN" "296-23648-6-ND"
+		(property "DKPN" "296-23648-1-ND"
 			(at 50.8 39.37 0)
 			(effects

Commit message: added level shift and breakout for UART/I2C
Parts:
- added H4: M3.5, lib_fp:MountingHole_3.5mm_Pad_Via, symbol lib_sch:MountingHole_Pad
- added J3: Conn_01x06_Pin, DS-Rectangular-Connectors:conn_01x06_254, symbol lib_sch:Conn_01x06_Pin
- added Q3, Q4: BSS138K, lib_fp:SOT23-3P95_237X112L50X40N, symbol lib_sch:NMOS_GSD
- added R6, R7, R8, R9: 4K7, lib_fp:CRCW0603, symbol lib_sch:R
- H1, H2: symbol Mechanical:MountingHole_Pad -> lib_sch:MountingHole_Pad
- H3: symbol Mechanical:MountingHole_Pad -> lib_sch:MountingHole_Pad; DKPN (none) -> 609-MDT420STD002TR-ND/4827-123A-NUT-42CT-ND; MPN (none) -> MDT420STD002/123A-NUT-42; Manufacturer (none) -> Amphenol ICC (FCI)/ATTEND Technology
Connections:
- net +1V8: now also Q3.1, Q4.1, R8.1, R9.1
- net +3V3: now also J3.1 (Pin_1), R6.1, R7.1
- net GND: now also H4.1, J3.6 (Pin_6)
- net SCL_3V3: now also J3.3 (Pin_3)
- net SDA_3V3: now also J3.2 (Pin_2)
- net RXD_1V8: now reaches J2.22 (UART_RXD)
- net RXD_1V8: now also Q3.2, R8.2
- net TXD_1V8: now reaches J2.32 (UART_TXD)
- net TXD_1V8: now also Q4.2, R9.2
- new net RXD_3V3: J3.5 (Pin_5), Q3.3, R6.2
- new net TXD_3V3: J3.4 (Pin_4), Q4.3, R7.2
- no-connect marks 75 -> 73
Other:
- note added: "Mounting Hardware Selection"
- moved on the sheet: J2
